Commit message: Its Alive

File: arm.urdf (robot description, URDF)
Before this commit: robot arm, 4 links, 3 joints
Links:
- link base_x: mass None -> 1
- link base_z: mass None -> 1
- link lower: mass None -> 1
- link upper: mass None -> 1

Commit message: not as alive

File: arm.urdf (robot description, URDF)
Before this commit: robot arm, 4 links, 3 joints
Links:
- link lower: geometry collision box size=.5 .5 1; visual box size=.5 .5 1
- link upper: geometry collision box size=.5 .5 1; visual box size=.5 .5 1
Joints:
- joint elbow: limit (none) -> lower=0 upper=0.1 effort=1000 velocity=1; origin xyz=0 0 3 rpy=0 0 0 -> xyz=0 0 1 rpy=0 0 0; type continuous -> revolute
- joint shoulder: limit (none) -> lower=0 upper=3.14 effort=1000 velocity=1; type continuous -> revolute

Commit message: arm goes wild at first but works

File: arm.urdf (robot description, URDF)
Before this commit: robot arm, 4 links, 3 joints
Links:
- link base_x: geometry visual sphere radius=0.025
- link base_z: geometry visual sphere radius=0.025
- link lower: mass 1 -> 0.3195; geometry collision box size=.381 .0254 0.0508; visual box size=.381 .0254 0.0508
- link upper: mass 1 -> 0.840; geometry collision box size=.5715 .0381 0.0762; visual box size=.5715 .0381 0.0762
Joints:
- joint elbow: axis 1 0 0 -> 0 1 0; limit lower=0 upper=0.1 effort=1000 velocity=1 -> (none); origin xyz=0 0 1 rpy=0 0 0 -> xyz=0.508 0 0 rpy=0 0 0; type revolute -> continuous
- joint shoulder: axis 1 0 0 -> 0 1 0; limit lower=0 upper=3.14 effort=1000 velocity=1 -> (none); type revolute -> continuous

Commit message: arm goes less wild but works - run "copy_pendulum_test.py"

File: arm.urdf (robot description, URDF)
Before this commit: robot arm, 4 links, 3 joints
Joints:
- joint elbow: limit (none) -> lower=-1.57 upper=1.57 effort=30 velocity=2.2; type continuous -> revolute
